File: hardware/kicad/smart_gas_meter_iot.kicad_sch (KiCad schematic)
At the start: 0 parts

Commit message: Replace graphical block concept with MIT reference-derived native ESP32-S3 schematic draft
Parts:
- added C1, C5: 10u, esp32-dev-boards:Capacitor_0805_2012, symbol Device:C
- added C2, C4: 100n, esp32-dev-boards:Capacitor_0805_2012, symbol Device:C
- added C3: 1u, esp32-dev-boards:Capacitor_0805_2012, symbol Device:C
- added D1: PWR, LED_SMD:LED_0805_2012Metric_Pad1.15x1.40mm_HandSolder, symbol Device:LED
- added D2: D, Diode_SMD:D_SMA, symbol Device:D
- added J1: ESP32-S3-DEVKITC-1-J1, esp32-dev-boards:ESP32-S3-DEVKITC-J1-mini, symbol esp32-dev-boards:ESP32-S3-DEVKITC-1-J1-mini
- added J2: ESP32-S3-DEVKITC-1-J2, esp32-dev-boards:ESP32-S3-DEVKITC-J2-mini, symbol esp32-dev-boards:ESP32-S3-DEVKITC-1-J2-mini
- added J3: ESP-Prog-ProgramCOM-RECV, $74th:BoxPinHeader_2x03_P1.27mm_Vertical, symbol $74th:ESP-Prog-ProgramCOM-RECV
- added J4: USB2.0_C_v3, $74th:USB-C-12-Pin-SMD, symbol $74th:USB2.0_C_v3
- added R1: 10k, esp32-dev-boards:Register_0805_2012, symbol Device:R
- added R2: 1k, esp32-dev-boards:Register_0805_2012, symbol Device:R
- added R3, R4: 5.1k, esp32-dev-boards:Register_0805_2012, symbol Device:R
- added SW1: RS, esp32-dev-boards:SKRPABE010, symbol Switch:SW_Push
- added SW2: BT, esp32-dev-boards:SKRPABE010, symbol Switch:SW_Push
- added U1: smart_gas_meter_iot, Espressif:ESP32-S3-WROOM-1, symbol Espressif:ESP32-S3-WROOM-1
- added U2: AMS1117-3.3, Package_TO_SOT_SMD:SOT-223-3_TabPin2, symbol Regulator_Linear:AMS1117-3.3
Connections:
- new net: D2.2 (A), J4.1 (VBUS)
- new net: J4.6 (CC2), R4.1
- new net: D1.2 (A), R2.1
- new net: J4.5 (CC1), R3.1
- new net +3V3: C1.1, C2.1, J1.2 (ESP_3V3), R1.2, R2.2, U1.2 (3V3), U2.2 (VO)
- new net +5V: C1.2, C2.2, C3.2, C4.1, C4.2, C5.1, C5.2, D1.1 (K), D2.1 (K), J1.21 (VCC_5V), J2.21 (GND), J3.2 (VCC), J3.4 (GND), J4.4 (GND), R3.2, R4.2, SW1.1, SW2.1, U1.1 (GND), U1.40 (GND), U1.41 (GND), U2.1 (GND), U2.3 (VI)
- new net CHIP_PU: C3.1, J1.3 (CHIP_PU), J3.1 (EN), R1.1, SW1.2, U1.3 (EN)
- new net GPIO0: J2.14 (GPIO0), J3.6 (IO0), SW2.2, U1.27 (GPIO0/BOOT)
- new net GPIO1: J2.4 (GPIO1), U1.39 (GPIO1/TOUCH1/ADC1_CH0)
- new net GPIO10: J1.16 (GPIO10), U1.18 (GPIO10/TOUCH10/ADC1_CH9/FSPICS0/FSPIIO4/SUBSPICS0)
- new net GPIO11: J1.17 (GPIO11), U1.19 (GPIO11/TOUCH11/ADC2_CH0/FSPID/FSPIIO5/SUBSPID)
- new net GPIO12: J1.18 (GPIO12), U1.20 (GPIO12/TOUCH12/ADC2_CH1/FSPICLK/FSPIIO6/SUBSPICLK)
- new net GPIO13: J1.19 (GPIO13), U1.21 (GPIO13/TOUCH13/ADC2_CH2/FSPIQ/FSPIIO7/SUBSPIQ)
- new net GPIO14: J1.20 (GPIO14), U1.22 (GPIO14/TOUCH14/ADC2_CH3/FSPIWP/FSPIDQS/SUBSPIWP)
- new net GPIO15: J1.8 (GPIO15), U1.8 (GPIO15/U0RTS/ADC2_CH4/XTAL_32K_P)
- new net GPIO16: J1.9 (GPIO16), U1.9 (GPIO16/U0CTS/ADC2_CH5/XTAL_32K_NH5)
- new net GPIO17: J1.10 (GPIO17), U1.10 (GPIO17/U1TXD/ADC2_CH6)
- new net GPIO18: J1.11 (GPIO18), U1.11 (GPIO18/U1RXD/ADC2_CH7/CLK_OUT3)
- new net GPIO19: J2.20 (GPIO19), J4.2 (D-), U1.13 (GPIO19/U1RTS/ADC2_CH8/CLK_OUT2/USB_D-)
- new net GPIO2: J2.5 (GPIO2), U1.38 (GPIO2/TOUCH2/ADC1_CH1)
- new net GPIO20: J2.19 (GPIO20), J4.3 (D+), U1.14 (GPIO20/U1CTS/ADC2_CH9/CLK_OUT1/USB_D+)
- new net GPIO21: J2.18 (GPIO21), U1.23 (GPIO21)
- new net GPIO3: J1.13 (GPIO3), U1.15 (GPIO3/TOUCH3/ADC1_CH2)
- new net GPIO35: J2.13 (GPIO35), U1.28 (SPIIO6/GPIO35/FSPID/SUBSPID)
- new net GPIO36: J2.12 (GPIO36), U1.29 (SPIIO7/GPIO36/FSPICLK/SUBSPICLK)
- new net GPIO37: J2.11 (GPIO37), U1.30 (SPIDQS/GPIO37/FSPIQ/SUBSPIQ)
- new net GPIO38: J2.10 (GPIO38), U1.31 (GPIO38/FSPIWP/SUBSPIWP)
- new net GPIO39: J2.9 (GPIO39), U1.32 (MTCK/GPIO39/CLK_OUT3/SUBSPICS1)
- new net GPIO4: J1.4 (GPIO4), U1.4 (GPIO4/TOUCH4/ADC1_CH3)
- new net GPIO40: J2.8 (GPIO40), U1.33 (MTDO/GPIO40/CLK_OUT2)
- new net GPIO41: J2.7 (GPIO41), U1.34 (MTDI/GPIO41/CLK_OUT1)
- new net GPIO42: J2.6 (GPIO42), U1.35 (MTMS/GPIO42)
- new net GPIO45: J2.15 (GPIO45), U1.26 (GPIO45)
- new net GPIO46: J1.14 (GPIO46), U1.16 (GPIO46)
- new net GPIO47: J2.17 (GPIO47), U1.24 (GPIO47/SPICLK_P/SUBSPICLK_P_DIFF)
- new net GPIO48: J2.16 (GPIO48), U1.25 (GPIO48/SPICLK_N/SUBSPICLK_N_DIFF)
- new net GPIO5: J1.5 (GPIO5), U1.5 (GPIO5/TOUCH5/ADC1_CH4)
- new net GPIO6: J1.6 (GPIO6), U1.6 (GPIO6/TOUCH6/ADC1_CH5)
- new net GPIO7: J1.7 (GPIO7), U1.7 (GPIO7/TOUCH7/ADC1_CH6)
- new net GPIO8: J1.12 (GPIO8), U1.12 (GPIO8/TOUCH8/ADC1_CH7/SUBSPICS1)
- new net GPIO9: J1.15 (GPIO9), U1.17 (GPIO9/TOUCH9/ADC1_CH8/FSPIHD/SUBSPIHD)
- new net U0RXD: J2.3 (U0RXD), J3.5 (RXD0), U1.36 (U0RXD/GPIO44/CLK_OUT2)
- new net U0TXD: J2.2 (U0TXD), J3.3 (TXD0), U1.37 (U0TXD/GPIO43/CLK_OUT1)
Other:
- note added: "Button"
- note added: "ESP32-S3 Module"
- note added: "Pinout"
- note added: "Power"
- note added: "Program Port"
- note added: "USB"
- note removed: "3V3 LOGIC REGULATOR ESP32-S3 rail Exact regulator TBD +3V3_LOGIC"
- note removed: "Draft functional sheet — symbols, pin-level wiring, power calculations, footprints and ERC remain to be completed."
- note removed: "ENGINEERING HOLD POINTS No native pin-level circuit finalized No ERC/DRC performed yet NOT FOR FABRICATION"
- note removed: "J2 — LAB PULSE Synthetic 3.3 V only series resistor + clamp pull-up; test point"
- note removed: "J3 — CELLULAR DAUGHTERBOARD UART + EN/RESET/STATUS SIM/RF per exact module docs SKU/operator/bands unconfirmed"
- note removed: "J4 — DEBUG HEADER GND / 3V3 / UART RESET / BOOT / TEST PADS"
- note removed: "OPTIONAL RTC / SPI FLASH Local queue + timekeeping Only after GPIO / retention review"
- note removed: "PROTECTED INPUT Fuse / TVS / reverse protection TBD +5V_SERVICE"
- note removed: "SEPARATE MODEM RAIL Peak-current budget required Never from MCU 3V3 Input / modem SKU TBD"
- note removed: "SMART GAS METER IoT — FUNCTIONAL BLOCK SCHEMATIC"
- note removed: "U1 — ESP32-S3-WROOM-1-N8 (proposed) Native USB D+/D−; EN/BOOT; local decoupling GPIO4: LAB_PULSE_IN; GPIO5: TAMPER_SW GPIO17/18: reserved modem UART (provisional)"
- note removed: "USB-C SERVICE INPUT 5 V only CC1/CC2 Rd + ESD J1 — exact part TBD"
- company: Smart Gas Meter IoT -> (none)
- title: Smart Gas Meter IoT — Engineering Schematic Draft -> ESP32-S3 Dev Board

Commit message: Correct module value and project title in native schematic draft
Parts:
- U1: value smart_gas_meter_iot -> ESP32-S3-WROOM-1
Other:
- title: ESP32-S3 Dev Board -> Smart Gas Meter IoT — ESP32-S3 carrier draft
Changed lines of the file:
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@@
   (paper "A4")
   (title_block
-    (title "ESP32-S3 Dev Board")
+    (title "Smart Gas Meter IoT — ESP32-S3 carrier draft")
     (rev "1.2.0")
   )
@@
       (effects (font (size 1.27 1.27)))
     )
-    (property "Value" "smart_gas_meter_iot" (at 94.615 25.4 0)
-      (effects (font (size 1.27 1.27)))
-    )
+    (property "Value" "ESP32-S3-WROOM-1" (at 94.615 25.4 0)
+      (effects (font (size 1.27 1.27)))
+    )

Commit message: Add engineering draft and laboratory safety status to schematic title block
Other:
- company: (none) -> Smart Gas Meter IoT
Changed lines of the file:
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@@
   (title_block
     (title "Smart Gas Meter IoT — ESP32-S3 carrier draft")
-    (rev "1.2.0")
+    (date "2026-10-21")
+    (rev "0.2-reference-derived")
+    (company "Smart Gas Meter IoT")
+    (comment 1 "ENGINEERING DRAFT — ERC and electrical review required")
+    (comment 2 "LOW-VOLTAGE LAB ONLY — synthetic pulse input; never connect to gas line")
   )
   (junction (at 259.08 35.56) (diameter 0) (color 0 0 0 0)
